Commit message: Rivz simulation build

File: src/arduinobot_description/urdf/arduinobot.urdf.xacro (robot description, xacro)
@@ -1 +1,36 @@
 <?xml version="1.0"?>
+<robot xmlns:xacro="http://www.ros.org/wiki/xacro" name="arduinobot">
+    <xacro:property name="PI" value="3.14159"/>
+    <xacro:property name="effort" value="30.0"/>
+    <xacro:property name="velocity" value="10.0"/>
+    <link name="world"/>
+    <!-- world center with basement -->
+    <link name="base_link">
+        <visual>
+            <origin rpy="0.0 0.0 0.0" xyz="-0.5 -0.5 0.0"/>
+            <geometry>
+                <mesh filename="package://arduinobot_description/meshes/basement.STL" scale="0.01 0.01 0.01"/>
+            </geometry>
+        </visual>
+    </link>
+    <joint name="virtual_joint" type="fixed">
+        <parent link="world"/>
+        <child link="base_link"/>
+        <origin rpy="0.0 0.0 0.0" xyz="0.0 0.0 0.0"/>
+    </joint>
+    <link name="base_plate">
+        <visual>
+            <origin xyz="-0.36 -0.4 -0.58" rpy="0 0 0"/>
+            <geometry>
+                <mesh filename="package://arduinobot_description/meshes/base_plate.STL" scale="0.01 0.01 0.01"/>
+            </geometry>
+        </visual>
+    </link>
+    <joint name="joint_1" type="revolute">
+        <parent link="base_link"/>
+        <child link="base_plate"/>
+        <origin xyz="0 0 0.307" rpy="0 0 0"/>
+        <axis xyz="0 0 1"/>
+        <limit lower="-${PI/2}" upper="${PI/2}" effort="${effort}" velocity="${velocity}"/>
+    </joint>
+</robot>

Commit message: world joint1 joint2

File: src/arduinobot_description/urdf/arduinobot.urdf.xacro (robot description, xacro)
@@ -34,3 +34,18 @@
         <limit lower="-${PI/2}" upper="${PI/2}" effort="${effort}" velocity="${velocity}"/>
     </joint>
+    <link name="forward_drive_arm">
+        <visual>
+            <origin xyz="0.22 0.07 -0.08" rpy="0 -${PI/2} ${PI/2}"/>
+            <geometry>
+                <mesh filename="package://arduinobot_description/meshes/forward_drive_arm.STL" scale="0.01 0.01 0.01"/>
+            </geometry>
+        </visual>
+    </link>
+    <joint name="joint_2" type="revolute">
+        <parent link="base_plate"/>
+        <child link="forward_drive_arm"/>
+        <origin xyz="-0.02 0 0.35" rpy="0 0 0"/>
+        <axis xyz="1 0 0"/>
+        <limit lower="-${PI/2}" upper="${PI/2}" effort="${effort}" velocity="${velocity}"/>
+    </joint>
 </robot>

Commit message: Rivz URDF finish

File: src/arduinobot_description/urdf/arduinobot.urdf.xacro (robot description, xacro)
@@ -4,4 +4,5 @@
     <xacro:property name="effort" value="30.0"/>
     <xacro:property name="velocity" value="10.0"/>
+    <!-- world -->
     <link name="world"/>
     <!-- world center with basement -->
@@ -19,4 +20,5 @@
         <origin rpy="0.0 0.0 0.0" xyz="0.0 0.0 0.0"/>
     </joint>
+    <!-- baseplate rotation -->
     <link name="base_plate">
         <visual>
@@ -34,4 +36,5 @@
         <limit lower="-${PI/2}" upper="${PI/2}" effort="${effort}" velocity="${velocity}"/>
     </joint>
+    <!-- forwardarm rotation -->
     <link name="forward_drive_arm">
         <visual>
@@ -49,3 +52,68 @@
         <limit lower="-${PI/2}" upper="${PI/2}" effort="${effort}" velocity="${velocity}"/>
     </joint>
+    <!-- horizontal_arm rotation  -->
+    <link name="horizontal_arm">
+        <visual>
+            <origin xyz="0.055 -0.43 -0.08" rpy="${PI/2} 0 ${PI/2}"/>
+            <geometry>
+                <mesh filename="package://arduinobot_description/meshes/horizontal_arm.STL" scale="0.01 0.01 0.01"/>
+            </geometry>
+        </visual>
+    </link>
+    <joint name="joint_3" type="revolute">
+        <parent link="forward_drive_arm"/>
+        <child link="horizontal_arm"/>
+        <origin xyz="-0.04 0.01 0.8" rpy="0 0 0"/>
+        <axis xyz="1 0 0"/>
+        <limit lower="-${PI/2}" upper="${PI/2}" effort="${effort}" velocity="${velocity}"/>
+    </joint>
+    <!-- claw support -->
+    <link name="claw_support">
+        <visual>
+            <origin xyz="0.16 -0.05 -0.130" rpy="0 0 ${PI/2}"/>
+            <geometry>
+                <mesh filename="package://arduinobot_description/meshes/claw_support.STL" scale="0.01 0.01 0.01"/>
+            </geometry>
+        </visual>
+    </link>
+    <joint name="horizontal_arm to claw_support" type="fixed">
+        <parent link="horizontal_arm"/>
+        <child link="claw_support"/>
+        <origin xyz="0.055 0.8 0" rpy="0 0 0"/>
+        <axis xyz="1 0 0"/>
+        <limit lower="-${PI/2}" upper="${PI/2}" effort="${effort}" velocity="${velocity}"/>
+    </joint>
+    <!-- gripper_left -->
+    <link name="gripper_left">
+        <visual>
+            <origin xyz="-0.04 0.47 +0.01" rpy="0 0 -${PI/2}"/>
+            <geometry>
+                <mesh filename="package://arduinobot_description/meshes/left_finger.STL" scale="0.01 0.01 0.01"/>
+            </geometry>
+        </visual>
+    </link>
+    <joint name="joint_4" type="revolute">
+        <parent link="claw_support"/>
+        <child link="gripper_left"/>
+        <origin xyz="-0.055 0.15 -0.1" rpy="0 0 0"/>
+        <axis xyz="0 0 1"/>
+        <limit lower="0" upper="${PI/6}" effort="${effort}" velocity="${velocity}"/>
+    </joint>
+    <!-- gripper_right -->
+    <link name="gripper_right">
+        <visual>
+            <origin xyz="-0.10 0.47 +0.01" rpy="0 0 -${PI/2}"/>
+            <geometry>
+                <mesh filename="package://arduinobot_description/meshes/right_finger.STL" scale="0.01 0.01 0.01"/>
+            </geometry>
+        </visual>
+    </link>
+    <joint name="joint_5" type="revolute">
+        <parent link="claw_support"/>
+        <child link="gripper_right"/>
+        <origin xyz="+0.125 0.15 -0.1" rpy="0 0 0"/>
+        <axis xyz="0 0 1"/>
+        <limit lower="-${PI/6}" upper="0" effort="${effort}" velocity="${velocity}"/>
+        <mimic joint="joint_4" multiplier="-1" offset="0"/>
+    </joint>
 </robot>
